File: SmartButton_rev3/button30mm_rev3.kicad_pcb (KiCad board)
At the start: 2 copper layers, 14.2 x 15.7 mm, 12 parts, among them J1 Conn_01x03_Pin, J2 B3B-XH-A, J3 Blade_LED, J4 Blade_LED, J5 Blade_SW, J6 Blade_SW, U1 PIC16F15213-I/SN

Commit message: Finished the layout
Parts:
- BR1: footprint Package_TO_SOT_SMD:SOT-143 -> library:SOT143_DIO
- moved U1 0.37 mm to (101.0, 63.2)
- moved BR1 0.35 mm to (95.1, 61.1), turned to 90 degrees
