File: SmartButton_rev3/button30mm_rev3.kicad_sch (KiCad schematic)
At the start: 12 parts, among them J1 Conn_01x03_Pin, J2 B3B-XH-A, J3 Blade_LED, J4 Blade_LED, J5 Blade_SW, J6 Blade_SW, U1 PIC16F15213-I/SN

Commit message: Finished the layout
Parts:
- BR1: footprint Package_TO_SOT_SMD:SOT-143 -> library:SOT143_DIO
Changed lines of the file:
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@@
 			)
 		)
-		(property "Footprint" "Package_TO_SOT_SMD:SOT-143"
+		(property "Footprint" "library:SOT143_DIO"
 			(at 218.44 85.09 0)
 			(effects
